Commit message: Modified files to simulate effort controller

File: urdf/practice_v3.xacro (robot description, xacro)
@@ -13,5 +13,5 @@
 			<child link="${prefix}_link"/>
 			<axis xyz="0 0 1"/>
-			<limit velocity="12.0" effort="0.4"/>
+			<limit velocity="12.0" effort="1.0"/>
 			<dynamics damping="0.1"/>
 		</joint>
@@ -19,8 +19,10 @@
 			<type>transmission_interface/SimpleTransmission</type>
 				<joint name="${prefix}_joint">
-					<hardwareInterface>hardware_interface/VelocityJointInterface</hardwareInterface>
+					<!-- <hardwareInterface>hardware_interface/EffortJointInterface</hardwareInterface> -->
+					<hardwareInterface>hardware_interface/EffortJointInterface</hardwareInterface>
 				</joint>
 				<actuator name="${prefix}_motor">
-					<hardwareInterface>hardware_interface/VelocityJointInterface</hardwareInterface>
+					<!-- <hardwareInterface>hardware_interface/EffortJointInterface</hardwareInterface> -->
+					<hardwareInterface>hardware_interface/EffortJointInterface</hardwareInterface>
 					<mechanicalReduction>1</mechanicalReduction>
 				</actuator>

Commit message: Modified for effort control

File: urdf/practice_v3.xacro (robot description, xacro)
@@ -13,5 +13,5 @@
 			<child link="${prefix}_link"/>
 			<axis xyz="0 0 1"/>
-			<limit velocity="12.0" effort="1.0"/>
+			<limit velocity="300.0" effort="10.0"/>
 			<dynamics damping="0.1"/>
 		</joint>
